File: Desktop Hardware Monitor/Desktop Hardware Monitor.kicad_pcb (KiCad board)
At the start: 2 copper layers, 38 parts, among them J1 USB_C_Receptacle_USB2.0, Q1 2N3904, Q2 2N3904, Q3 2N3904, Q4 2N3904, Q5 2N3904, Q6 2N3904, SW1 Reset Switch, U1 ATmega328-P, U10 SM420561N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

Commit message: Update PCB Files
Parts:
- added ?: , , F.Cu at (189.1, 68.3)
- added ?: , , F.Cu at (188.4, 132.3)
- added ?: , , F.Cu at (90.5, 132.4)
- added J2: Conn_01x02_Female, Connector_PinHeader_2.54mm:PinHeader_1x02_P2.54mm_Vertical, F.Cu at (94.5, 90.7)
- added J3: Conn_01x02_Female, Connector_PinHeader_2.54mm:PinHeader_1x02_P2.54mm_Vertical, F.Cu at (97.1, 86.9)
- added REF**: MountingHole_2.2mm_M2_DIN965_Pad, MountingHole:MountingHole_2.2mm_M2_DIN965_Pad, F.Cu at (90.5, 68.3)
- moved U6 109.0 mm to (169.5, 127.2), turned to 90 degrees
- moved U5 104.4 mm to (158.2, 121.2), turned to -90 degrees
- moved U4 83.9 mm to (138.6, 121.2), turned to -90 degrees
- moved Q2 64.2 mm to (151.7, 89.2)
- moved U10 61.1 mm to (148.1, 83.9)
- moved C1 54.9 mm to (98.2, 112.8), turned to 180 degrees
- moved Q6 52.6 mm to (154.3, 96.0)
- moved Q5 52.5 mm to (140.7, 96.0)
- moved Q3 52.2 mm to (124.5, 89.1)
- moved Q4 52.1 mm to (127.1, 95.9)
- moved U8 51.8 mm to (173.5, 78.3)
- moved R_D7 51.5 mm to (148.5, 87.5), turned to -90 degrees
- moved J1 50.5 mm to (97.4, 68.3)
- moved U14 49.7 mm to (148.1, 116.5)
- moved R_D3 49.5 mm to (157.5, 97.7)
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Connections:
- U7 pad 1: unconnected-(U7-Pad1) -> GND
- U7 pad 2: unconnected-(U7-Pad2) -> VCC
- U7 pad 3: unconnected-(U7-Pad3) -> SCL
- U7 pad 4: unconnected-(U7-Pad4) -> SDA
Routing:
- net SDA: track 0.00 -> 89.4 mm, vias 0 -> 3
- net SCL: track 0.00 -> 88.5 mm, vias 0 -> 3
- net VCC: track 94.9 -> 156.1 mm
- net Net-(R_D1-Pad2): track 76.4 -> 121.9 mm, vias 0 -> 1
- net Net-(RG1-Pad2): track 153.2 -> 112.6 mm, vias 2 -> 0
- net Net-(U4-Pad14): track 51.2 -> 18.3 mm
- net Net-(R_D4-Pad2): track 22.2 -> 54.4 mm, vias 0 -> 1
- net RST: track 15.6 -> 47.5 mm
- net A0: track 16.6 -> 46.0 mm
- net Net-(U4-Pad13): track 42.7 -> 17.4 mm
- net E: track 28.8 -> 4.07 mm
- net DP: track 10.5 -> 33.8 mm
- net G: track 36.6 -> 58.3 mm, vias 0 -> 1
- net CLK: track 27.6 -> 49.0 mm
- net F: track 34.1 -> 54.7 mm
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- added copper zone on B.Cu, net GND
- added copper zone on F.Cu, net GND
Other:
- board outline added: 106 x 71.3 mm
- board text added: "RXD"
- board text added: "SCL"
- board text added: "SDA"
- board text added: "TXD"
