File: Desktop Hardware Monitor/Desktop Hardware Monitor.kicad_sch (KiCad schematic)
At the start: 39 parts, among them J1 USB_C_Receptacle_USB2.0, Q2 2N3904, Q3 2N3904, Q4 2N3904, Q5 2N3904, Q6 2N3904, SW1 Reset Switch, U1 ATmega328-P, U10 SM420561N, U11 SM420561N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

Commit message: Update PCB Files
Parts:
- added J2, J3: (no value), symbol Connector:Conn_01x02_Female
- added J4: (no value), symbol Connector_Generic_Shielded:Conn_01x04_Shielded
- C0, C1: footprint (none) -> Capacitor_THT:C_Disc_D5.1mm_W3.2mm_P5.00mm
- J1: footprint (none) -> Connector_PinHeader_2.54mm:PinHeader_1x05_P2.54mm_Vertical
- Q1: value (none) -> 2N3904; footprint (none) -> Package_TO_SOT_THT:TO-92_Inline
- RG1, R_A1, R_B1, R_C1, R_D1, R_D5, R_DP1, R_E1, R_F1: value (none) -> 1K; footprint (none) -> Resistor_THT:R_Axial_DIN0207_L6.3mm_D2.5mm_P10.16mm_Horizontal
- R_D2, R_D3, R_D4, R_D6, R_D7: footprint (none) -> Resistor_THT:R_Axial_DIN0207_L6.3mm_D2.5mm_P10.16mm_Horizontal
- U12: value (none) -> SM420561N; footprint (none) -> Display_7Segment:7SegmentLED_LTS6760_LTS6780
- U2: value (none) -> TCA9548a
- U4: value (none) -> 74LS138; footprint (none) -> Package_DIP:DIP-16_W7.62mm_Socket
- U5: value (none) -> 74LS04; footprint (none) -> Package_DIP:DIP-14_W7.62mm_Socket
- U8: footprint (none) -> WS2812B:IC2_Display_4_Pin
- X1: footprint (none) -> Crystal:Crystal_HC49-4H_Vertical
Connections:
- net +5V: now also SW1.3 (K)
- net RXD: now also J2.1 (Pin_1)
- net SCL: now also J3.2 (Pin_2)
- net SDA: now also J3.1 (Pin_1)
- net TXD: now also J2.2 (Pin_2)
Other:
- note added: "RXD/TXD Breakout"
- note added: "SDA/SCL Breakout"
